File: axis-cover/axis-cover.kicad_sch (KiCad schematic)
At the start: 7 parts

Commit message: Update
Parts:
- H1, H2, H3: now left out of the parts list
Other:
- moved on the sheet: ICON1
Changed lines of the file:
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@@
 	(title_block
 		(title "V2 axis")
-		(date "2023-01-09")
-		(rev "1")
+		(date "2024-07-19")
+		(rev "2")
 		(company "Versio Duo")
 		(comment 1 "cover")
@@
 			)
 		)
+		(property "Sim.Enable" "0"
+			(at 177.8 137.16 0)
+			(effects
+				(font
+					(size 1.27 1.27)
+				)
+				(hide yes)
+			)
+		)
 		(instances
 			(project "axis-cover"
@@
 			)
 		)
+		(property "Sim.Enable" "0"
+			(at 130.81 123.19 0)
+			(effects
+				(font
+					(size 1.27 1.27)
+				)
+				(hide yes)
+			)
+		)
 		(instances
 			(project "axis-cover"
@@
 		(unit 1)
 		(exclude_from_sim no)
-		(in_bom yes)
+		(in_bom no)
 		(on_board yes)
 		(dnp no)
@@
 			)
 		)
+		(property "Sim.Enable" "0"
+			(at 129.54 78.74 0)
+			(effects
+				(font
+					(size 1.27 1.27)
+				)
+				(hide yes)
+			)
+		)
 		(pin "1"
 		)
@@
 			)
 		)
+		(property "Sim.Enable" "0"
+			(at 152.4 137.16 0)
+			(effects
+				(font
+					(size 1.27 1.27)
+				)
+				(hide yes)
+			)
+		)
 		(instances
 			(project "axis-cover"
@@
 		(unit 1)
 		(exclude_from_sim no)
-		(in_bom yes)
+		(in_bom no)
 		(on_board yes)
 		(dnp no)
@@
 			)
 		)
+		(property "Sim.Enable" "0"
+			(at 130.81 105.41 0)
+			(effects
+				(font
+					(size 1.27 1.27)
+				)
+				(hide yes)
+			)
+		)
 		(instances
 			(project "axis-cover"
@@
 			)
 		)
+		(property "Sim.Enable" "0"
+			(at 132.08 135.89 0)
+			(effects
+				(font
+					(size 1.27 1.27)
+				)
+				(hide yes)
+			)
+		)
 		(instances
 			(project "axis-cover"
@@
 		(unit 1)
 		(exclude_from_sim no)
-		(in_bom yes)
+		(in_bom no)
 		(on_board yes)
 		(dnp no)
@@
 			(at 129.54 87.63 0)
 			(effects
+				(font
+					(size 1.27 1.27)
+				)
+				(hide yes)
+			)
+		)
+		(property "Sim.Enable" "0"
+			(at 129.54 87.63 0)
+			(effects

Commit message: Update
Parts:
- H2, H3: footprint V2_Mechanical:Mounting_Hole_2mm_Pad_5.2mm -> V2_Mechanical:MountingHole_2mm_Pad_5.2mm
Changed lines of the file:
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@@
 (kicad_sch
-	(version 20231120)
+	(version 20250114)
 	(generator "eeschema")
-	(generator_version "8.0")
+	(generator_version "9.0")
 	(paper "A4")
 	(title_block
 		(title "V2 axis")
-		(date "2024-07-19")
-		(rev "2")
+		(date "2025-10-30")
+		(rev "3")
 		(company "Versio Duo")
 		(comment 1 "cover")
@@
 			)
 		)
-		(property "Footprint" "V2_Mechanical:Mounting_Hole_2mm_Pad_5.2mm"
+		(property "Footprint" "V2_Mechanical:MountingHole_2mm_Pad_5.2mm"
 			(at 119.38 78.74 0)
 			(effects
@@
 			)
 		)
-		(property "Footprint" "V2_Mechanical:Mounting_Hole_2mm_Pad_5.2mm"
+		(property "Footprint" "V2_Mechanical:MountingHole_2mm_Pad_5.2mm"
 			(at 119.38 87.63 0)
 			(effects
@@
 		)
 	)
+	(embedded_fonts no)
 )
